File: 12V_power_supply_tryout.sch (KiCad schematic (older format))
At the start: 14 parts, among them J9 Barrel_Jack_Switch, U6 XL4015

Commit message: update,
Parts:
- gave numbers to parts that had none: 1
Changed lines of the file:
@@
 $EndComp
 $Comp
-L Connector_Generic:Conn_01x02 J?
+L Connector_Generic:Conn_01x02 J1
 U 1 1 5C06C762
 P 10400 3750
-F 0 "J?" H 10500 3750 50  0000 L CNN
+F 0 "J1" H 10500 3750 50  0000 L CNN
 F 1 "Conn_01x02" H 10500 3650 50  0000 L CNN
 F 2 "Connector_PinHeader_2.54mm:PinHeader_1x02_P2.54mm_Vertical" H 10400 3750 50  0001 C CNN
@@
 $EndComp
 $Comp
-L power:+12V #PWR?
+L power:+12V #PWR0101
 U 1 1 5C06C7BE
 P 10000 3650
-F 0 "#PWR?" H 10000 3500 50  0001 C CNN
+F 0 "#PWR0101" H 10000 3500 50  0001 C CNN
 F 1 "+12V" H 10015 3823 50  0000 C CNN
 F 2 "" H 10000 3650 50  0001 C CNN
@@
 $EndComp
 $Comp
-L power:GND #PWR?
+L power:GND #PWR0102
 U 1 1 5C06C842
 P 10000 4050
-F 0 "#PWR?" H 10000 3800 50  0001 C CNN
+F 0 "#PWR0102" H 10000 3800 50  0001 C CNN
 F 1 "GND" H 10050 3850 50  0000 C CNN
 F 2 "" H 10000 4050 50  0001 C CNN
